Commit message: start training

File: source/amazing/amazing/assets/urdf/15_Test1.urdf (robot description, URDF)
Before this commit: robot 15_Test1, 15 links, 14 joints
Links:
- link FL1_1: mass 4.143447954247557 -> 0.5; geometry collision mesh filename=../meshes/FL1_1.stl scale=0.001 0.001 0.001; visual mesh filename=../meshes/FL1_1.stl scale=0.001 0.001 0.001
- link FL2_1: mass 2.510112518506589 -> 0.5; geometry collision mesh filename=../meshes/FL2_1.stl scale=0.001 0.001 0.001; visual mesh filename=../meshes/FL2_1.stl scale=0.001 0.001 0.001
- link FR1_1: mass 4.143448003039892 -> 0.5; geometry collision mesh filename=../meshes/FR1_1.stl scale=0.001 0.001 0.001; visual mesh filename=../meshes/FR1_1.stl scale=0.001 0.001 0.001
- link FR2_1: mass 2.5101125185065984 -> 0.5; geometry collision mesh filename=../meshes/FR2_1.stl scale=0.001 0.001 0.001; visual mesh filename=../meshes/FR2_1.stl scale=0.001 0.001 0.001
- link SL_1: mass 2.0840497794889576 -> 0.5; geometry collision mesh filename=../meshes/SL_1.stl scale=0.001 0.001 0.001; visual mesh filename=../meshes/SL_1.stl scale=0.001 0.001 0.001
- link SR_1: mass 2.0840498282812847 -> 0.5; geometry collision mesh filename=../meshes/SR_1.stl scale=0.001 0.001 0.001; visual mesh filename=../meshes/SR_1.stl scale=0.001 0.001 0.001
- link T1_1: mass 0.1090568786472829 -> 0.5; geometry collision mesh filename=../meshes/T1_1.stl scale=0.001 0.001 0.001; visual mesh filename=../meshes/T1_1.stl scale=0.001 0.001 0.001
- link T2_1: mass 1.186572261162841 -> 0.5; geometry collision mesh filename=../meshes/T2_1.stl scale=0.001 0.001 0.001; visual mesh filename=../meshes/T2_1.stl scale=0.001 0.001 0.001
- link T3_1: mass 1.0987230693934555 -> 0.5  ; geometry collision mesh filename=../meshes/T3_1.stl scale=0.001 0.001 0.001; visual mesh filename=../meshes/T3_1.stl scale=0.001 0.001 0.001
- link T4_1: mass 0.505290360000207 -> 0.1; geometry collision mesh filename=../meshes/T4_1.stl scale=0.001 0.001 0.001; visual mesh filename=../meshes/T4_1.stl scale=0.001 0.001 0.001
- link T5_1: mass 0.691185972108562 -> 0.1; geometry collision mesh filename=../meshes/T5_1.stl scale=0.001 0.001 0.001; visual mesh filename=../meshes/T5_1.stl scale=0.001 0.001 0.001
- link T6_1: mass 0.021934067900310803 -> 0.05; geometry collision mesh filename=../meshes/T6_1.stl scale=0.001 0.001 0.001; visual mesh filename=../meshes/T6_1.stl scale=0.001 0.001 0.001
- link WL_1: mass 0.49375167072519255 -> 0.5; geometry collision mesh filename=../meshes/WL_1.stl scale=0.001 0.001 0.001; visual mesh filename=../meshes/WL_1.stl scale=0.001 0.001 0.001
- link WR_1: mass 3.8759486776453422 -> 0.5; geometry collision mesh filename=../meshes/WR_1.stl scale=0.001 0.001 0.001; visual mesh filename=../meshes/WR_1.stl scale=0.001 0.001 0.001
- link base_link: mass 19.811169104366787 -> 0.5; geometry collision mesh filename=../meshes/base_link.stl scale=0.001 0.001 0.001; visual mesh filename=../meshes/base_link.stl scale=0.001 0.001 0.001
